File: 1_ega/3_esquematico_pcb/ega-sch/ega-sch.kicad_sch (KiCad schematic)
At the start: 54 parts, among them J1 Encoder, J2 TFT_Display, J3 MCP4725, J4 DS3231, J6 V+, J7 Ventrada, Q1 IRFZ44, SW1 SW_Push, U1 ESP32-S3-DEVKITC-1-N16R8V, U2 LM7805_TO220, U3 LM358

Commit message: Add: Agrego ultima version ega
Connections:
- net I2C1_SDA: now reaches U1.J1_10 (GPIO17)
- net I2C1_SCL: now reaches U1.J1_11 (GPIO18)
- net UART_TX: now reaches U1.J3_2 (U0TXD/GPIO43)
- net UART_RX: now reaches U1.J3_3 (U0RXD/GPIO44)
Other:
- note added: "EGA - CARGA ELECTRONICA"
Changed lines of the file:
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@@
 	(generator_version "9.0")
 	(paper "A4")
+	(text "EGA - CARGA ELECTRONICA"
+		(exclude_from_sim no)
+		(at 229.108 173.736 0)
+		(effects
+			(font
+				(size 2.54 2.54)
+			)
+		)
+	)
 	(text "10ohm"
 		(exclude_from_sim no)
@@
 	(wire
 		(pts
+			(xy 86.36 68.58) (xy 93.98 68.58)
+		)
+		(stroke
+			(width 0)
+			(type default)
+		)
+	)
+	(wire
+		(pts
 			(xy 29.21 121.92) (xy 33.02 121.92)
 		)
@@
 	(wire
 		(pts
+			(xy 36.83 78.74) (xy 40.64 78.74)
+		)
+		(stroke
+			(width 0)
+			(type default)
+		)
+	)
+	(wire
+		(pts
 			(xy 27.94 97.79) (xy 33.02 97.79)
 		)
@@
 	(wire
 		(pts
+			(xy 36.83 76.2) (xy 40.64 76.2)
+		)
+		(stroke
+			(width 0)
+			(type default)
+		)
+	)
+	(wire
+		(pts
 			(xy 171.45 75.565) (xy 178.435 75.565)
 		)
@@
 	(wire
 		(pts
+			(xy 86.36 71.12) (xy 93.98 71.12)
+		)
+		(stroke
+			(width 0)
+			(type default)
+		)
+	)
+	(wire
+		(pts
 			(xy 186.69 132.08) (xy 189.23 132.08)
 		)
@@
 			(width 0)
 			(type default)
+		)
+	)
+	(label "UART_TX"
+		(at 93.98 68.58 0)
+		(effects
+			(font
+				(size 1.27 1.27)
+			)
+			(justify left bottom)
+		)
+	)
+	(label "UART_RX"
+		(at 93.98 71.12 0)
+		(effects
+			(font
+				(size 1.27 1.27)
+			)
+			(justify left bottom)
+		)
+	)
+	(label "I2C1_SDA"
+		(at 36.83 76.2 180)
+		(effects
+			(font
+				(size 1.27 1.27)
+			)
+			(justify right bottom)
 		)
 	)
@@
 		)
 	)
+	(label "I2C1_SCL"
+		(at 36.83 78.74 180)
+		(effects
+			(font
+				(size 1.27 1.27)
+			)
+			(justify right bottom)
+		)
+	)
